File: BSPD/BSPD/BSPD.kicad_sch (KiCad schematic)
At the start: 37 parts, among them J1 430450626, K1 AZ943-1CH-12DE, U3 74HC1G08GW_125, U4 74HC1G02GW_125, U5 LTC6994CS6-1-TRMPBF, U6 DRDC3105F-7, U7 LD1117S50TR_SOT223

Commit message: Configured footprints and set board outline.
All footprints have been assigned to the components, and the board size and it's mounting holes have been set up in the pcb editor.
Parts:
- removed J1: 430450626, CONN_SD-43045-009_06_MOL, symbol Molex_430450626:430450626
- added J1: 430450613, Molex_430450613:CONN_SD-43045-005_06_MOL, symbol Molex_430450613:430450613
- C1, C2, C3, C4, C5, C6: footprint (none) -> CL10A104K:CAP_CL10_SAM
- D1, D2, D3, D4, D5, D6, D7, D8: footprint (none) -> CMD17_21VGD:LED0805N_CML
- K1: footprint AZ943-1CH_AMZ -> AZ943_1CH_12DE:AZ943-1CH_AMZ
- R1, R10, R19, R2, R20, R21, R3, R4, R5, R6, R7, R8, R9: footprint (none) -> Resistor_SMD:R_0603_1608Metric_Pad0.98x0.95mm_HandSolder
- RV1, RV2: footprint (none) -> PV36W103C01B00:RES3_PV36W103C01B00_BRN
- U3, U4: footprint TSSOP5_SOT353-1_NEX -> Package_TO_SOT_SMD:SOT-353_SC-70-5
- U5: footprint TSOT-23_S6_LIT -> LTC6994:TSOT-23_S6_LIT
- U6: footprint SOT23_DIO -> DRDC3105:SOT23_DIO
- U8: footprint (none) -> Package_TO_SOT_SMD:SOT-23-8
Connections:
- net +12V: now also J1.1
- net Brake Sense: now also J1.2
- net Current Sense: now also J1.3
- net GND: now also J1.4
- net Shutdown In: now also J1.6
- net Shutdown Out: now also J1.5
Changed lines of the file:
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@@
 	)
 	(label "Shutdown In"
-		(at 248.92 43.18 180)
+		(at 248.92 50.8 180)
 		(fields_autoplaced yes)
 		(effects
@@
 	)
 	(label "Shutdown Out"
-		(at 248.92 50.8 180)
+		(at 248.92 48.26 180)
 		(fields_autoplaced yes)
 		(effects
@@
 	)
 	(label "Current Sense"
-		(at 248.92 48.26 180)
+		(at 248.92 43.18 180)
 		(fields_autoplaced yes)
 		(effects
@@
 			)
 		)
-		(property "Footprint" ""
+		(property "Footprint" "CMD17_21VGD:LED0805N_CML"
 			(at 120.65 171.45 0)
 			(effects
@@
 			)
 		)
-		(property "Footprint" "TSSOP5_SOT353-1_NEX"
+		(property "Footprint" "Package_TO_SOT_SMD:SOT-353_SC-70-5"
 			(at 141.986 49.53 0)
 			(effects
@@
 			)
 		)
-		(property "Footprint" ""
+		(property "Footprint" "CMD17_21VGD:LED0805N_CML"
 			(at 135.89 171.45 0)
 			(effects
@@
 			)
 		)
-		(property "Footprint" ""
+		(property "Footprint" "CMD17_21VGD:LED0805N_CML"
 			(at 44.45 171.45 0)
 			(effects
@@
 			)
 		)
-		(property "Footprint" "SOT23_DIO"
+		(property "Footprint" "DRDC3105:SOT23_DIO"
 			(at 195.58 118.11 0)
 			(effects
@@
 			)
 		)
-		(property "Footprint" "TSOT-23_S6_LIT"
+		(property "Footprint" "LTC6994:TSOT-23_S6_LIT"
 			(at 135.89 118.11 0)
 			(effects
@@
 			)
 		)
-		(property "Footprint" ""
+		(property "Footprint" "Resistor_SMD:R_0603_1608Metric_Pad0.98x0.95mm_HandSolder"
 			(at 48.26 81.28 0)
 			(effects
@@
 			)
 		)
-		(property "Footprint" ""
+		(property "Footprint" "CMD17_21VGD:LED0805N_CML"
 			(at 105.41 171.45 0)
 			(effects
@@
 			)
 		)
-		(property "Footprint" ""
+		(property "Footprint" "Resistor_SMD:R_0603_1608Metric_Pad0.98x0.95mm_HandSolder"
 			(at 67.31 81.28 0)
 			(effects
@@
 			)
 		)
-		(property "Footprint" ""
+		(property "Footprint" "CMD17_21VGD:LED0805N_CML"
 			(at 91.44 171.45 0)
 			(effects
@@
 			)
 		)
-		(property "Footprint" ""
+		(property "Footprint" "CL10A104K:CAP_CL10_SAM"
 			(at 156.21 137.4648 0)
 			(effects
@@
 			)
 		)
-		(property "Footprint" ""
+		(property "Footprint" "CMD17_21VGD:LED0805N_CML"
 			(at 73.66 171.45 0)
 			(effects
@@
 	)
 	(symbol
+		(lib_id "Molex_430450613:430450613")
+		(at 248.92 38.1 0)
+		(unit 1)
+		(exclude_from_sim no)
+		(in_bom yes)
+		(on_board yes)
+		(dnp no)
+		(fields_autoplaced yes)
+		(property "Reference" "J1"
+			(at 262.89 43.1799 0)
+			(effects
+				(font
+					(size 1.524 1.524)
+				)
+				(justify left)
+			)
+		)
+		(property "Value" "430450613"
+			(at 262.89 45.7199 0)
+			(effects
+				(font
+					(size 1.524 1.524)
+				)
+				(justify left)
+			)
+		)
+		(property "Footprint" "Molex_430450613:CONN_SD-43045-005_06_MOL"
+			(at 248.92 38.1 0)
+			(effects
+				(font
+					(size 1.27 1.27)
+					(italic yes)
+				)
+				(hide yes)
+			)
+		)
+		(property "Datasheet" "430450613"
+			(at 248.92 38.1 0)
+			(effects
+				(font
+					(size 1.27 1.27)
+					(italic yes)
+				)
+				(hide yes)
+			)
+		)
+		(property "Description" ""
+			(at 248.92 38.1 0)
+			(effects
+				(font
+					(size 1.27 1.27)
+				)
+				(hide yes)
+			)
+		)
+		(pin "2"
+		)
+		(pin "3"
+		)
+		(pin "6"
+		)
+		(pin "5"
+		)
+		(pin "1"
+		)
+		(pin "4"
+		)
+		(instances
+			(project ""
+				(path "/e182f3fc-f710-48d1-be81-2e1aaca2fe5e"
+					(reference "J1")
+					(unit 1)
+				)
+			)
+		)
+	)
+	(symbol
 		(lib_id "power:GND")
 		(at 160.02 57.15 0)
@@
 			)
 		)
-		(property "Footprint" ""
+		(property "Footprint" "CMD17_21VGD:LED0805N_CML"
 			(at 30.48 171.45 0)
 			(effects
@@
 			)
 		)
-		(property "Footprint" ""
+		(property "Footprint" "Resistor_SMD:R_0603_1608Metric_Pad0.98x0.95mm_HandSolder"
 			(at 103.632 162.56 90)
 			(effects
@@
 			)
 		)
-		(property "Footprint" ""
+		(property "Footprint" "CL10A104K:CAP_CL10_SAM"
 			(at 178.7652 45.72 0)
 			(effects
@@
 			)
 		)
-		(property "Footprint" "AZ943-1CH_AMZ"
+		(property "Footprint" "AZ943_1CH_12DE:AZ943-1CH_AMZ"
 			(at 232.41 115.57 0)
 			(effects
@@
 			)
 		)
-		(property "Footprint" ""
+		(property "Footprint" "Resistor_SMD:R_0603_1608Metric_Pad0.98x0.95mm_HandSolder"
 			(at 118.872 162.56 90)
 			(effects
@@
 			)
 		)
-		(property "Footprint" ""
+		(property "Footprint" "PV36W103C01B00:RES3_PV36W103C01B00_BRN"
 			(at 67.31 49.53 0)
 			(effects
@@
 			)
 		)
-		(property "Footprint" ""
+		(property "Footprint" "Resistor_SMD:R_0603_1608Metric_Pad0.98x0.95mm_HandSolder"
 			(at 132.842 128.27 90)
 			(effects
@@
 			)
 		)
-		(property "Footprint" ""
+		(property "Footprint" "Resistor_SMD:R_0603_1608Metric_Pad0.98x0.95mm_HandSolder"
 			(at 42.672 162.56 90)
 			(effects
@@
 			)
 		)
-		(property "Footprint" "TSSOP5_SOT353-1_NEX"
+		(property "Footprint" "Package_TO_SOT_SMD:SOT-353_SC-70-5"
 			(at 99.314 102.362 0)
 			(effects
@@
 			)
 		)
-		(property "Footprint" ""
+		(property "Footprint" "CL10A104K:CAP_CL10_SAM"
 			(at 120.65 112.0648 0)
 			(effects
@@
 			)
 		)
-		(property "Footprint" ""
+		(property "Footprint" "Resistor_SMD:R_0603_1608Metric_Pad0.98x0.95mm_HandSolder"
 			(at 89.662 162.56 90)
 			(effects
@@
 			)
 		)
-		(property "Footprint" ""
+		(property "Footprint" "CL10A104K:CAP_CL10_SAM"
 			(at 125.73 38.4048 0)
 			(effects
@@
 			)
 		)
-		(property "Footprint" ""
+		(property "Footprint" "PV36W103C01B00:RES3_PV36W103C01B00_BRN"
 			(at 48.26 49.53 0)
 			(effects
@@
 			)
 		)
-		(property "Footprint" ""
+		(property "Footprint" "Resistor_SMD:R_0603_1608Metric_Pad0.98x0.95mm_HandSolder"
 			(at 134.112 162.56 90)
 			(effects
@@
 			)
 		)
-		(property "Footprint" ""
+		(property "Footprint" "Resistor_SMD:R_0603_1608Metric_Pad0.98x0.95mm_HandSolder"
 			(at 28.702 162.56 90)
 			(effects
@@
 			)
 		)
-		(property "Footprint" ""
+		(property "Footprint" "CL10A104K:CAP_CL10_SAM"
 			(at 158.75 54.9148 0)
 			(effects
@@
 			)
 		)
-		(property "Footprint" ""
+		(property "Footprint" "Resistor_SMD:R_0603_1608Metric_Pad0.98x0.95mm_HandSolder"
 			(at 71.882 162.56 90)
 			(effects
@@
 			)
 		)
-		(property "Footprint" ""
+		(property "Footprint" "Resistor_SMD:R_0603_1608Metric_Pad0.98x0.95mm_HandSolder"
 			(at 172.212 123.19 90)
 			(effects
@@
 	)
 	(symbol
-		(lib_id "Molex_430450626:430450626")
-		(at 248.92 38.1 0)
-		(unit 1)
-		(exclude_from_sim no)
-		(in_bom yes)
-		(on_board yes)
-		(dnp no)
-		(fields_autoplaced yes)
-		(property "Reference" "J1"
-			(at 262.89 43.1799 0)
-			(effects
-				(font
-					(size 1.524 1.524)
-				)
-				(justify left)
-			)
-		)
-		(property "Value" "430450626"
-			(at 262.89 45.7199 0)
-			(effects
-				(font
-					(size 1.524 1.524)
-				)
-				(justify left)
-			)
-		)
-		(property "Footprint" "CONN_SD-43045-009_06_MOL"
-			(at 248.92 38.1 0)
-			(effects
-				(font
-					(size 1.27 1.27)
-					(italic yes)
-				)
-				(hide yes)
-			)
-		)
-		(property "Datasheet" "430450626"
-			(at 248.92 38.1 0)
-			(effects
-				(font
-					(size 1.27 1.27)
-					(italic yes)
-				)
-				(hide yes)
-			)
-		)
-		(property "Description" ""
-			(at 248.92 38.1 0)
-			(effects
-				(font
-					(size 1.27 1.27)
-				)
-				(hide yes)
-			)
-		)
-		(pin "2"
-		)
-		(pin "4"
-		)
-		(pin "1"
-		)
-		(pin "5"
-		)
-		(pin "6"
-		)
-		(pin "3"
-		)
-		(instances
-			(project ""
-				(path "/e182f3fc-f710-48d1-be81-2e1aaca2fe5e"
-					(reference "J1")
-					(unit 1)
-				)
-			)
-		)
-	)
-	(symbol
 		(lib_id "Device:R")
 		(at 57.15 162.56 0)
@@
 			)
 		)
-		(property "Footprint" ""
+		(property "Footprint" "Resistor_SMD:R_0603_1608Metric_Pad0.98x0.95mm_HandSolder"
 			(at 55.372 162.56 90)
 			(effects
@@
 			)
 		)
-		(property "Footprint" ""
+		(property "Footprint" "CL10A104K:CAP_CL10_SAM"
 			(at 206.7052 45.72 0)
 			(effects
@@
 			)
 		)
-		(property "Footprint" ""
+		(property "Footprint" "CMD17_21VGD:LED0805N_CML"
 			(at 57.15 171.45 0)
 			(effects
@@
 			)
 		)
-		(property "Footprint" ""
+		(property "Footprint" "Resistor_SMD:R_0603_1608Metric_Pad0.98x0.95mm_HandSolder"
 			(at 172.212 130.81 90)
 			(effects
@@
 			)
 		)
-		(property "Footprint" ""
+		(property "Footprint" "Package_TO_SOT_SMD:SOT-23-8"
 			(at 85.09 66.04 0)
 			(effects

Commit message: Layout started and component changes
The footprints have all be chosen and the linear regulator was swapped out.
Parts:
- removed D5, D6, D7, D8: LED, CMD17_21VGD:LED0805N_CML, symbol Device:LED
- removed R10, R19, R20, R9: 300, Resistor_SMD:R_0603_1608Metric_Pad0.98x0.95mm_HandSolder, symbol Device:R
- removed U7: LD1117S50TR_SOT223, Package_TO_SOT_SMD:SOT-223-3_TabPin2, symbol Regulator_Linear:LD1117S50TR_SOT223
- added U7: UA78M05CDCYR, Package_TO_SOT_SMD:SOT-223-3_TabPin2, symbol UA78M05CDCYR:UA78M05CDCYR
- C2: value 100n -> 0.33u
- C3: value 10u -> 0.1u
Connections:
- net +12V: now also U7.1 (IN)
- net +5V: now also U7.3 (OUT)
- net BSP: now also U4.1 (B); no longer U4.2 (A)
- net Circuit Fault: now also U4.2 (A); no longer U4.1 (B)
- net GND: now also U7.2 (GND)
Other:
- moved on the sheet: D1, D2, D3, D4, R1, R21, R3, R8
